Commit message: model mostly OK, inertia added

File: catkin_ws/src/rov_hil/urdf/macros.xacro (robot description, xacro)
@@ -1,72 +1,122 @@
 <?xml version="1.0" ?>
 <robot name="x3_rov_macros" xmlns:xacro="http://www.ros.org/wiki/xacro">
-   <!-- fin -->
-    <xacro:macro name="fin" params="suffix parent_link origin_xyz rad len">
-        <link name="Lfin_${suffix}">
-            <collision>
-                <origin rpy="0 ${pi/2} 0" xyz="${-len/4} 0 0"/>
-                <geometry>
-                    <cylinder radius="${rad}" length="${len/2}"/>
-                </geometry>
-            </collision>
-            <visual>
-                <origin rpy="0 ${pi/2} 0" xyz="${-len/4} 0 0"/>
-                <geometry>
-                    <cylinder radius="${rad}" length="${len/2}"/>
-                </geometry>
-                <material name="black"/>
-            </visual>
-        </link>
-        <joint name="Jfin_${suffix}" type="fixed">
-            <parent link="${parent_link}"/>
-            <child link="Lfin_${suffix}"/>
-            <origin xyz="${origin_xyz}" rpy="0 0 0"/>
-            <axis xyz="0 0 0"/>
-	    </joint>
-    </xacro:macro>
-    <!-- propeller -->
-    <xacro:macro name="prop" params="suffix parent_link origin_xyz rad len mirror">
-        <link name="Lprop_conn_${suffix}">
-            <collision>
-                <origin rpy="0 ${pi/2} 0" xyz="${-len/4} 0 0"/>
-                <geometry>
-                    <cylinder radius="${rad * 2/3}" length="${len/2}"/>
-                </geometry>
-            </collision>
-            <visual>
-                <origin rpy="0 ${pi/2} 0" xyz="${-len/4} 0 0"/>
-                <geometry>
-                    <cylinder radius="${rad * 2/3}" length="${len/2}"/>
-                </geometry>
-                <material name="black"/>
-            </visual>
-        </link>
-        <joint name="Jprop_conn_${suffix}" type="fixed">
-            <parent link="${parent_link}"/>
-            <child link="Lprop_conn_${suffix}"/>
-            <origin xyz="${origin_xyz}" rpy="0 0 0"/>
-            <axis xyz="0 0 0"/>
-        </joint>
-        <link name="Lprop_body_${suffix}">
-            <collision>
-                <origin rpy="0 ${pi/2} 0" xyz="${-len/4} 0 0"/>
-                <geometry>
-                    <cylinder radius="${rad}" length="${len/2}"/>
-                </geometry>
-            </collision>
-            <visual>
-                <origin rpy="0 ${pi/2} 0" xyz="${-len/4} 0 0"/>
-                <geometry>
-                    <cylinder radius="${rad}" length="${len/2}"/>
-                </geometry>
-                <material name="black"/>
-            </visual>
-        </link>
-        <joint name="Jprop_body_${suffix}" type="fixed">
-            <parent link="Lprop_conn_${suffix}"/>
-            <child link="Lprop_body_${suffix}"/>
-            <origin xyz="${-len/2} ${mirror * rad * 1/3} 0" rpy="0 0 0"/>
-            <axis xyz="0 0 0"/>
-        </joint>
-    </xacro:macro>
+	<!-- * * * inertial calculations * * * -->
+	<!-- sources: -->
+	<!-- https://github.com/ros-industrial/universal_robot/blob/06d8b9e2f5f86aa54f9f2845f11edbc84e2f951e/ur_description/urdf/ur10.urdf.xacro#L12-L20 -->
+	<!-- https://answers.ros.org/question/293281/using-xacro-to-automate-inertial-calculations-sequencefloat-error/ -->
+	<!-- cuboid -->
+	<xacro:macro name="cuboid_inertial" params="*origin mass length width height">
+    <inertial>
+      <mass value="${mass}"/>
+			<xacro:insert_block name="origin" />
+      <inertia
+				ixx="${0.83 * mass * (width  + height)}" ixy="0.0" ixz="0.0"
+				iyy="${0.83 * mass * (length + height)}" iyz="0.0"
+				izz="${0.83 * mass * (width  + length)}"
+			/>
+    </inertial>
+  </xacro:macro>
+	<!-- cylinder -->
+	<xacro:macro name="cylinder_inertial" params="*origin mass radius length">
+    <inertial>
+      <mass value="${mass}" />
+			<xacro:insert_block name="origin" />
+      <inertia
+				ixx="${0.0833333 * mass * (3 * radius * radius + length * length)}" ixy="0.0" ixz="0.0"
+        iyy="${0.0833333 * mass * (3 * radius * radius + length * length)}" iyz="0.0"
+        izz="${0.5 * mass * radius * radius}"
+			/>
+    </inertial>
+  </xacro:macro>
+	<!-- * * * macros for creating links * * * -->
+	<!-- create fin and attach to parent -->
+	<xacro:macro name="fin" params="suffix parent_link origin_xyz mass radius length">
+		<link name="Lfin_${suffix}">
+			<xacro:cylinder_inertial
+				mass="${mass}"
+				radius="${radius}"
+				length="${length}"
+			>
+				<origin xyz="${-length/2} 0 0" rpy="0 ${pi/2} 0"/>
+			</xacro:cylinder_inertial>
+			<collision>
+				<origin xyz="${-length/2} 0 0" rpy="0 ${pi/2} 0"/>
+				<geometry>
+					<cylinder radius="${radius}" length="${length}"/>
+				</geometry>
+			</collision>
+			<!-- <visual>
+				<origin rpy="0 ${pi/2} 0" xyz="${-length/2} 0 0"/>
+				<geometry>
+					<cylinder radius="${radius}" length="${length}"/>
+				</geometry>
+				<material name="black"/>
+			</visual> -->
+		</link>
+		<joint name="Jfin_${suffix}" type="fixed">
+			<parent link="${parent_link}"/>
+			<child link="Lfin_${suffix}"/>
+			<origin xyz="${origin_xyz}" rpy="0 0 0"/>
+			<axis xyz="0 0 0"/>
+		</joint>
+	</xacro:macro>
+	<!-- create propeller and attach to parent -->
+	<xacro:macro name="prop" params="suffix parent_link origin_xyz mass radius length mirror">
+		<link name="Lprop_conn_${suffix}">
+			<xacro:cylinder_inertial
+				mass="${mass * 1/3}"
+				radius="${radius * 2/3}"
+				length="${length/2}"
+			>
+				<origin xyz="${-length/4} 0 0" rpy="0 ${pi/2} 0"/>
+			</xacro:cylinder_inertial>
+			<collision>
+				<origin xyz="${-length/4} 0 0" rpy="0 ${pi/2} 0"/>
+				<geometry>
+					<cylinder radius="${radius * 2/3}" length="${length/2}"/>
+				</geometry>
+			</collision>
+			<!-- <visual>
+				<origin xyz="${-length/4} 0 0" rpy="0 ${pi/2} 0" />
+				<geometry>
+					<cylinder radius="${radius * 2/3}" length="${length/2}"/>
+				</geometry>
+				<material name="black"/>
+			</visual> -->
+		</link>
+		<joint name="Jprop_conn_${suffix}" type="fixed">
+			<parent link="${parent_link}"/>
+			<child link="Lprop_conn_${suffix}"/>
+			<origin xyz="${origin_xyz}" rpy="0 0 0"/>
+			<axis xyz="0 0 0"/>
+		</joint>
+		<link name="Lprop_body_${suffix}">
+			<xacro:cylinder_inertial
+				mass="${mass * 2/3}"
+				radius="${radius}"
+				length="${length/2}"
+			>
+				<origin xyz="${-length/4} 0 0" rpy="0 ${pi/2} 0"/>
+			</xacro:cylinder_inertial>
+			<collision>
+				<origin xyz="${-length/4} 0 0" rpy="0 ${pi/2} 0"/>
+				<geometry>
+					<cylinder radius="${radius}" length="${length/2}"/>
+				</geometry>
+			</collision>
+			<!-- <visual>
+				<origin xyz="${-length/4} 0 0 rpy="0 ${pi/2} 0""/>
+				<geometry>
+					<cylinder radius="${radius}" length="${length/2}"/>
+				</geometry>
+				<material name="black"/>
+			</visual> -->
+		</link>
+		<joint name="Jprop_body_${suffix}" type="fixed">
+			<parent link="Lprop_conn_${suffix}"/>
+			<child link="Lprop_body_${suffix}"/>
+			<origin xyz="${-length/2} ${mirror * radius * 1/8} 0" rpy="0 0 0"/>
+			<axis xyz="0 0 0"/>
+		</joint>
+	</xacro:macro>
 </robot>

File: catkin_ws/src/rov_hil/urdf/x3_v1.xacro (robot description, xacro)
@@ -1,74 +1,86 @@
 <?xml version="1.0"?>
 <robot name="x3_rov" xmlns:xacro="http://www.ros.org/wiki/xacro">
-    <!-- includes -->
-    <xacro:include filename="$(find rov_hil)/urdf/materials.xacro" />
-    <xacro:include filename="$(find rov_hil)/urdf/macros.xacro" />
-    <!-- properties -->
-    <xacro:property name="x3_length" value="0.485" />
-    <xacro:property name="x3_width" value="0.257" />
-    <xacro:property name="x3_height" value="0.354" />
+	<!-- includes -->
+	<xacro:include filename="$(find rov_hil)/urdf/materials.xacro" />
+	<xacro:include filename="$(find rov_hil)/urdf/macros.xacro" />
+	<!-- properties/variables -->
+	<xacro:property name="x3_length" value="0.485" />	<!-- m  -->
+	<xacro:property name="x3_width"  value="0.257" /> <!-- m  -->
+	<xacro:property name="x3_height" value="0.354" /> <!-- m  -->
+	<xacro:property name="x3_mass"   value="9" />     <!-- kg -->
+	<!-- calculations are based roughly on volume distribution -->
+	<xacro:property name="x3_m_main" value="${x3_mass * 0.66}" />
+	<xacro:property name="x3_m_fin"  value="${x3_mass * 0.14}" />
+	<xacro:property name="x3_m_prop" value="${x3_mass * 0.03}" />
 	<!-- * * * Link Definitions * * * -->
-    <link name="Lhitbox">
-        <collision>
-            <origin rpy="0 0 0" xyz="0 0 0"/>
-            <geometry>
-                <box size="${x3_length} ${x3_width} ${x3_height}"/>
-            </geometry>
-        </collision>
-        <visual>
-            <origin rpy="0 0 0" xyz="0 0 0"/>
-            <geometry>
-                <box size="${x3_length} ${x3_width} ${x3_height}"/>
-                <!-- <mesh filename="package://my_cobot/models/joint1.dae"/> -->
-            </geometry>
-            <material name="grey_transparent"/>
-        </visual>
+	<!-- Dummy link to suppress warnings about root link inertia -->
+	<link name="dummy">
 	</link>
-    <link name="Lmain">
-        <collision>
-            <origin rpy="0 0 0" xyz="${x3_length * 3/16} 0 0"/>
-            <geometry>
-                <box size="${x3_length*5/8} ${x3_width * 3/5} ${x3_height}"/>
-            </geometry>
-        </collision>
-        <visual>
-            <origin rpy="0 0 0" xyz="${x3_length * 3/16} 0 0"/>
-            <geometry>
-                <box size="${x3_length*5/8} ${x3_width * 3/5} ${x3_height}"/>
-            </geometry>
-            <material name="black"/>
-        </visual>
+	<link name="Lmain">
+		<xacro:cuboid_inertial
+			mass="${x3_m_main}"
+			length="${x3_length}"
+			width="${x3_width}"
+			height="${x3_height}"
+		>
+			<origin xyz="${x3_length * 3/16} 0 0" rpy="0 0 0"/>
+		</xacro:cuboid_inertial>
+		<collision>
+			<origin xyz="${x3_length * 3/16} 0 0" rpy="0 0 0"/>
+			<geometry>
+				<box size="${x3_length*5/8} ${x3_width * 3/5} ${x3_height}"/>
+			</geometry>
+		</collision>
+		<visual>
+			<!-- <origin rpy="0 0 0" xyz="${x3_length * 3/16} 0 0"/> -->
+			<origin xyz="0 0 0" rpy="0 0 0"/>
+			<geometry>
+				<!-- <box size="${x3_length*5/8} ${x3_width * 3/5} ${x3_height}"/> -->
+				<mesh filename="package://rov_hil/models/x3_low_poly_smoothed.dae"/>
+			</geometry>
+			<material name="grey_transparent"/>
+		</visual>
 	</link>
-    <joint name="Jmain" type="fixed">
-    	<parent link="Lhitbox"/>
-    	<child link="Lmain"/>
-        <origin xyz="0 0 0" rpy="0 0 0"/>
-        <axis xyz="0 0 0"/>
+	<joint name="dummy_joint" type="fixed">
+		<parent link="dummy"/>
+		<child link="Lmain"/>
 	</joint>
-    <xacro:fin
-        suffix="top"
-        parent_link="Lmain"
-        origin_xyz="0 0 ${x3_height*(1/2 - 1/6)}"
-        rad="${x3_height * 1/6}"
-        len="${x3_length}"/>
-    <xacro:fin
-        suffix="bot"
-        parent_link="Lmain"
-        origin_xyz="0 0 ${-x3_height*(1/2 - 1/6)}"
-        rad="${x3_height * 1/6}"
-        len="${x3_length}"/>
-    <xacro:prop
-        suffix="left"
-        parent_link="Lmain"
-        origin_xyz="0 ${x3_width * 3/10} 0"
-        rad="${x3_height * 1/9}"
-        len="${x3_length * 1/3}"
-        mirror="1"/>
-    <xacro:prop
-        suffix="right"
-        parent_link="Lmain"
-        origin_xyz="0 ${-(x3_width * 3/10)} 0"
-        rad="${x3_height * 1/9}"
-        len="${x3_length * 1/3}"
-        mirror="-1"/>
+	<!-- top fin -->
+	<xacro:fin
+		suffix="top"
+		parent_link="Lmain"
+		origin_xyz="0 0 ${x3_height*(1/2 - 1/6)}"
+		mass="${x3_m_fin}"
+		radius="${x3_height * 1/6}"
+		length="${x3_length/2}"
+	/>
+	<!-- bottom fin -->
+	<xacro:fin
+		suffix="bot"
+		parent_link="Lmain"
+		origin_xyz="0 0 ${-x3_height*(1/2 - 1/6)}"
+		mass="${x3_m_fin}"
+		radius="${x3_height * 1/6}"
+		length="${x3_length/2}"
+	/>
+	<!-- left propeller -->
+	<xacro:prop
+		suffix="left"
+		parent_link="Lmain"
+		origin_xyz="0 ${x3_width * 3/10} 0"
+		mass="${x3_m_prop}"
+		radius="${x3_height * 1/8}"
+		length="${x3_length * 1/3}"
+		mirror="1"
+	/>
+	<!-- right propeller -->
+	<xacro:prop
+		suffix="right"
+		parent_link="Lmain"
+		origin_xyz="0 ${-(x3_width * 3/10)} 0"
+		mass="${x3_m_prop}"
+		radius="${x3_height * 1/8}"
+		length="${x3_length * 1/3}"
+		mirror="-1"
+	/>
 </robot>
