Commit message: copied uuv ws, gazebo simulation OK!

File: catkin_ws/src/rov_hil/urdf/macros.xacro (robot description, xacro)
@@ -1,20 +1,11 @@
 <?xml version="1.0" ?>
 <robot name="x3_rov_macros" xmlns:xacro="http://www.ros.org/wiki/xacro">
+	<!-- properties/variables -->
+	<xacro:arg name="debug" default="0"/>
+	<xacro:arg name="namespace" default="x3_rov"/>
+	<xacro:arg name="inertial_reference_frame" default="world"/>
 	<!-- * * * inertial calculations * * * -->
-	<!-- sources: -->
+	<!-- source: -->
 	<!-- https://github.com/ros-industrial/universal_robot/blob/06d8b9e2f5f86aa54f9f2845f11edbc84e2f951e/ur_description/urdf/ur10.urdf.xacro#L12-L20 -->
-	<!-- https://answers.ros.org/question/293281/using-xacro-to-automate-inertial-calculations-sequencefloat-error/ -->
-	<!-- cuboid -->
-	<xacro:macro name="cuboid_inertial" params="*origin mass length width height">
-    <inertial>
-      <mass value="${mass}"/>
-			<xacro:insert_block name="origin" />
-      <inertia
-				ixx="${0.83 * mass * (width  + height)}" ixy="0.0" ixz="0.0"
-				iyy="${0.83 * mass * (length + height)}" iyz="0.0"
-				izz="${0.83 * mass * (width  + length)}"
-			/>
-    </inertial>
-  </xacro:macro>
 	<!-- cylinder -->
 	<xacro:macro name="cylinder_inertial" params="*origin mass radius length">
@@ -23,5 +14,5 @@
 			<xacro:insert_block name="origin" />
       <inertia
-				ixx="${0.0833333 * mass * (3 * radius * radius + length * length)}" ixy="0.0" ixz="0.0"
+		ixx="${0.0833333 * mass * (3 * radius * radius + length * length)}" ixy="0.0" ixz="0.0"
         iyy="${0.0833333 * mass * (3 * radius * radius + length * length)}" iyz="0.0"
         izz="${0.5 * mass * radius * radius}"
@@ -31,6 +22,6 @@
 	<!-- * * * macros for creating links * * * -->
 	<!-- create fin and attach to parent -->
-	<xacro:macro name="fin" params="suffix parent_link origin_xyz mass radius length">
-		<link name="Lfin_${suffix}">
+	<xacro:macro name="x3_fin" params="suffix parent_link origin_xyz mass radius length">
+		<link name="$(arg namespace)/fin_${suffix}_link">
 			<xacro:cylinder_inertial
 				mass="${mass}"
@@ -46,22 +37,22 @@
 				</geometry>
 			</collision>
-			<!-- <visual>
+			<visual>
 				<origin rpy="0 ${pi/2} 0" xyz="${-length/2} 0 0"/>
 				<geometry>
-					<cylinder radius="${radius}" length="${length}"/>
+					<cylinder radius="1e-5" length="1e-5"/>
 				</geometry>
 				<material name="black"/>
-			</visual> -->
-		</link>
-		<joint name="Jfin_${suffix}" type="fixed">
+			</visual>
+		</link>
+		<joint name="$(arg namespace)/fin_${suffix}_joint" type="fixed">
 			<parent link="${parent_link}"/>
-			<child link="Lfin_${suffix}"/>
+			<child link="$(arg namespace)/fin_${suffix}_link"/>
 			<origin xyz="${origin_xyz}" rpy="0 0 0"/>
 			<axis xyz="0 0 0"/>
 		</joint>
 	</xacro:macro>
-	<!-- create propeller and attach to parent -->
-	<xacro:macro name="prop" params="suffix parent_link origin_xyz mass radius length mirror">
-		<link name="Lprop_conn_${suffix}">
+	<!-- create thruster housing and attach to parent -->
+	<xacro:macro name="x3_thruster" params="suffix parent_link origin_xyz mass radius length mirror">
+		<link name="$(arg namespace)/thruster_conn_${suffix}_link">
 			<xacro:cylinder_inertial
 				mass="${mass * 1/3}"
@@ -77,19 +68,19 @@
 				</geometry>
 			</collision>
-			<!-- <visual>
+			<visual>
 				<origin xyz="${-length/4} 0 0" rpy="0 ${pi/2} 0" />
 				<geometry>
-					<cylinder radius="${radius * 2/3}" length="${length/2}"/>
+					<cylinder radius="1e-5" length="1e-5"/>
 				</geometry>
 				<material name="black"/>
-			</visual> -->
-		</link>
-		<joint name="Jprop_conn_${suffix}" type="fixed">
+			</visual>
+		</link>
+		<joint name="$(arg namespace)/thruster_conn_${suffix}_joint" type="fixed">
 			<parent link="${parent_link}"/>
-			<child link="Lprop_conn_${suffix}"/>
+			<child link="$(arg namespace)/thruster_conn_${suffix}_link"/>
 			<origin xyz="${origin_xyz}" rpy="0 0 0"/>
 			<axis xyz="0 0 0"/>
 		</joint>
-		<link name="Lprop_body_${suffix}">
+		<link name="$(arg namespace)/thruster_body_${suffix}_link">
 			<xacro:cylinder_inertial
 				mass="${mass * 2/3}"
@@ -105,18 +96,172 @@
 				</geometry>
 			</collision>
-			<!-- <visual>
-				<origin xyz="${-length/4} 0 0 rpy="0 ${pi/2} 0""/>
-				<geometry>
-					<cylinder radius="${radius}" length="${length/2}"/>
+			<visual>
+				<origin xyz="${-length/4} 0 0" rpy="0 ${pi/2} 0"/>
+				<geometry>
+					<cylinder radius="1e-5" length="1e-5"/>
 				</geometry>
 				<material name="black"/>
-			</visual> -->
-		</link>
-		<joint name="Jprop_body_${suffix}" type="fixed">
-			<parent link="Lprop_conn_${suffix}"/>
-			<child link="Lprop_body_${suffix}"/>
+			</visual>
+		</link>
+		<joint name="$(arg namespace)/thruster_body_${suffix}_joint" type="fixed">
+			<parent link="$(arg namespace)/thruster_conn_${suffix}_link"/>
+			<child link="$(arg namespace)/thruster_body_${suffix}_link"/>
 			<origin xyz="${-length/2} ${mirror * radius * 1/8} 0" rpy="0 0 0"/>
 			<axis xyz="0 0 0"/>
 		</joint>
 	</xacro:macro>
+	<!-- camera macro - based off of uuv camera snippet with some modifications -->
+	<xacro:macro name="x3_camera" params="parent_link suffix *origin">
+		<link name="$(arg namespace)/camera${suffix}_link">
+			<xacro:box_inertial
+				mass="1e-4"
+				x="1e-4"
+				y="1e-4"
+				z="1e-4"
+			>
+			<origin xyz="0 0 0" rpy="0 0 0"/>
+			</xacro:box_inertial>
+			<visual>
+				<origin xyz="0 0 0" rpy="0 0 0"/>
+				<geometry>
+				<box size="1e-4 1e-4 1e-4"/>
+				</geometry>
+			</visual>
+			<collision>
+				<origin xyz="0 0 0" rpy="0 0 0"/>
+				<geometry>
+				<box size="1e-4 1e-4 1e-4"/>
+				</geometry>
+			</collision>
+		</link>
+		<joint name="$(arg namespace)/camera${suffix}_joint" type="revolute">
+			<parent link="${parent_link}"/>
+			<child link="$(arg namespace)/camera${suffix}_link"/>
+			<xacro:insert_block name="origin" />
+			<axis xyz="0 1 0"/>
+			<limit effort="1e-6" lower="${-pi/6}" upper="${pi/6}" velocity="0.5"/>
+		</joint>
+		<transmission name="$(arg namespace)/camera${suffix}/trans">
+			<type>transmission_interface/SimpleTransmission</type>
+			<joint name="$(arg namespace)/camera${suffix}_joint">
+				<hardwareInterface>hardware_interface/EffortJointInterface</hardwareInterface>
+			</joint>
+			<actuator name="$(arg namespace)/camera${suffix}/motor">
+				<hardwareInterface>hardware_interface/EffortJointInterface</hardwareInterface>
+				<mechanicalReduction>1</mechanicalReduction>
+			</actuator>
+		</transmission>
+		<gazebo reference="$(arg namespace)/camera${suffix}_link">
+			<sensor type="camera" name="camera${suffix}">
+				<update_rate>30</update_rate>
+				<camera name="camera${suffix}">
+				<vertical_fov>115</vertical_fov>
+				<image>
+					<width>1920</width>
+					<height>1080</height>
+					<format>R8G8B8</format>
+				</image>
+				<clip>
+					<near>0.05</near>
+					<far>3000</far>
+				</clip>
+				<noise>
+					<type>gaussian</type>
+					<mean>0.0</mean>
+					<stddev>0.02</stddev>
+				</noise>
+				</camera>
+				<plugin name="camera${suffix}_controller" filename="libgazebo_ros_camera.so">
+				<updateRate>30</updateRate>
+				<cameraName>$(arg namespace)/camera${suffix}</cameraName>
+				<frameName>$(arg namespace)/camera${suffix}_link</frameName>
+				<hackBaseline>0.07</hackBaseline>
+				<distortionK1>0.0</distortionK1>
+				<distortionK2>0.0</distortionK2>
+				<distortionK3>0.0</distortionK3>
+				<distortionT1>0.0</distortionT1>
+				<distortionT2>0.0</distortionT2>
+				<attenuationR>0.0</attenuationR>
+				<attenuationG>0.0</attenuationG>
+				<attenuationB>0.0</attenuationB>
+				<backgroundR>0</backgroundR>
+				<backgroundG>0</backgroundG>
+				<backgroundB>0</backgroundB>
+				<imageTopicName>image_raw</imageTopicName>
+				<!-- required for ros depth cam -->
+				<!-- <pointCloudTopicName>image_cloud</pointCloudTopicName>
+				<depthImageTopicName>image_depth</depthImageTopicName>
+				<depthImageCameraInfoTopicName>image_depth_info</depthImageCameraInfoTopicName>
+				<pointCloudCutoff>10.0</pointCloudCutoff> -->
+				</plugin>
+			</sensor>
+		</gazebo>
+	</xacro:macro>
+	<!-- hydrodynamic_model -->
+	<xacro:macro name="rov_hydro_model" params="parent_link mass length width height cob neutrally_buoyant">
+		<gazebo>
+			<plugin name="uuv_plugin" filename="libuuv_underwater_object_ros_plugin.so">
+				<!-- Hydro parameters for the vehicle-->
+				<fluid_density>1028.0</fluid_density>
+				<flow_velocity_topic>hydrodynamics/current_velocity</flow_velocity_topic>
+				<debug>$(arg debug)</debug>
+				<link name="${parent_link}">
+					<neutrally_buoyant>${neutrally_buoyant}</neutrally_buoyant>
+					<volume>${mass/1028}</volume>
+					<box>
+						<width>${width}</width>
+						<length>${length}</length>
+						<height>${height}</height>
+					</box>
+					<center_of_buoyancy>${cob}</center_of_buoyancy>
+					<hydrodynamic_model>
+						<type>fossen</type>
+						<added_mass>
+						<!-- based on values from rexrov but tweaked -->
+						<!-- not accurate at all currently -->
+						 400    0    0     0    0    0
+						   0  500    0     0    0    0
+						   0    0 1600     6    0    0
+						   0    0    0   500    0    0
+						   0    0    0     0  800    0
+						   0    0    0     0    0  200
+						 <!-- 770    0    0     0    0    0
+						   0 1200    0     0    0    0
+						   0    0 3600     6    0    0
+						   0    0    0   530    0    0
+						   0    0    0     0  840    0
+						   0    0    0     0    0  220 -->
+						</added_mass>
+						<!-- Linear damping: see p.31 in Berg2012 -->
+						<linear_damping>
+						 -50  -50  -100 -200 -200 -150
+						 <!-- -70  -65 -700  -260 -300 -100 -->
+						</linear_damping>
+						<!-- Non-linear damping: see p.30 in Berg2012 -->
+						<quadratic_damping>
+						-740 -990 -1200 -400 -500 -400
+						</quadratic_damping>
+					</hydrodynamic_model>
+				</link>
+			</plugin>
+		</gazebo>
+	</xacro:macro>
+	<!-- Thruster macro -->
+	<!-- Common values, colors, converstion, standard shapes/inertia etc.
+		Dependency for the thruster_snippets.xacro-->
+	<xacro:include filename="$(find uuv_descriptions)/urdf/common.urdf.xacro"/>
+	<xacro:include filename="$(find uuv_gazebo_ros_plugins)/urdf/thruster_snippets.xacro"/>
+	<!-- thruster model -->
+	<xacro:property name="thruster_mesh_file" value="file://$(find rov_hil)/models/x3_low_poly_propeller.dae"/>
+	<xacro:macro name="thruster_macro" params="thruster_id *origin">
+		<xacro:thruster_module_first_order_basic_fcn_macro
+			namespace="$(arg namespace)"
+			thruster_id="${thruster_id}"
+			mesh_filename="${thruster_mesh_file}"
+			dyn_time_constant="0.05"
+			rotor_constant="0.00025"
+			>
+			<xacro:insert_block name="origin"/>
+		</xacro:thruster_module_first_order_basic_fcn_macro>
+	</xacro:macro>
 </robot>

File: catkin_ws/src/rov_hil/urdf/x3_v1.xacro (robot description, xacro)
@@ -2,85 +2,139 @@
 <robot name="x3_rov" xmlns:xacro="http://www.ros.org/wiki/xacro">
 	<!-- includes -->
-	<xacro:include filename="$(find rov_hil)/urdf/materials.xacro" />
-	<xacro:include filename="$(find rov_hil)/urdf/macros.xacro" />
-	<!-- properties/variables -->
-	<xacro:property name="x3_length" value="0.485" />	<!-- m  -->
-	<xacro:property name="x3_width"  value="0.257" /> <!-- m  -->
-	<xacro:property name="x3_height" value="0.354" /> <!-- m  -->
-	<xacro:property name="x3_mass"   value="9" />     <!-- kg -->
-	<!-- calculations are based roughly on volume distribution -->
-	<xacro:property name="x3_m_main" value="${x3_mass * 0.66}" />
-	<xacro:property name="x3_m_fin"  value="${x3_mass * 0.14}" />
-	<xacro:property name="x3_m_prop" value="${x3_mass * 0.03}" />
-	<!-- * * * Link Definitions * * * -->
-	<!-- Dummy link to suppress warnings about root link inertia -->
-	<link name="dummy">
-	</link>
-	<link name="Lmain">
-		<xacro:cuboid_inertial
-			mass="${x3_m_main}"
-			length="${x3_length}"
-			width="${x3_width}"
-			height="${x3_height}"
-		>
-			<origin xyz="${x3_length * 3/16} 0 0" rpy="0 0 0"/>
-		</xacro:cuboid_inertial>
-		<collision>
-			<origin xyz="${x3_length * 3/16} 0 0" rpy="0 0 0"/>
-			<geometry>
-				<box size="${x3_length*5/8} ${x3_width * 3/5} ${x3_height}"/>
-			</geometry>
-		</collision>
-		<visual>
-			<!-- <origin rpy="0 0 0" xyz="${x3_length * 3/16} 0 0"/> -->
-			<origin xyz="0 0 0" rpy="0 0 0"/>
-			<geometry>
-				<!-- <box size="${x3_length*5/8} ${x3_width * 3/5} ${x3_height}"/> -->
-				<mesh filename="package://rov_hil/models/x3_low_poly_smoothed.dae"/>
-			</geometry>
-			<material name="grey_transparent"/>
-		</visual>
-	</link>
-	<joint name="dummy_joint" type="fixed">
-		<parent link="dummy"/>
-		<child link="Lmain"/>
-	</joint>
-	<!-- top fin -->
-	<xacro:fin
-		suffix="top"
-		parent_link="Lmain"
-		origin_xyz="0 0 ${x3_height*(1/2 - 1/6)}"
-		mass="${x3_m_fin}"
-		radius="${x3_height * 1/6}"
-		length="${x3_length/2}"
-	/>
-	<!-- bottom fin -->
-	<xacro:fin
-		suffix="bot"
-		parent_link="Lmain"
-		origin_xyz="0 0 ${-x3_height*(1/2 - 1/6)}"
-		mass="${x3_m_fin}"
-		radius="${x3_height * 1/6}"
-		length="${x3_length/2}"
-	/>
-	<!-- left propeller -->
-	<xacro:prop
-		suffix="left"
-		parent_link="Lmain"
-		origin_xyz="0 ${x3_width * 3/10} 0"
-		mass="${x3_m_prop}"
-		radius="${x3_height * 1/8}"
-		length="${x3_length * 1/3}"
-		mirror="1"
-	/>
-	<!-- right propeller -->
-	<xacro:prop
-		suffix="right"
-		parent_link="Lmain"
-		origin_xyz="0 ${-(x3_width * 3/10)} 0"
-		mass="${x3_m_prop}"
-		radius="${x3_height * 1/8}"
-		length="${x3_length * 1/3}"
-		mirror="-1"
-	/>
+	<!-- "Dummy" base link to eliminate root link inertia warning -->
+  <link name="$(arg namespace)/dummy_link"/>
+ <!-- base_link according to ROS conventions: x forward, z up -->
+ <link name="$(arg namespace)/base_link">
+   <inertial>
+     <mass value="1862.87"/>
+     <origin xyz="0 0 0"/>
+     <inertia ixx="52.39" ixy="1.44" ixz="33.41" iyy="79.20" iyz="2.6" izz="69.23"/>
+   </inertial>
+   <visual>
+     <origin xyz="0 0 0" rpy="0 0 1.5708"/>
+     <geometry>
+       <mesh filename="package://smilodon_description/meshes/smilodon_nologo_visual.dae" scale="1 1 1"/>
+     </geometry>
+   </visual>
+   <collision>
+     <origin xyz="0 0 0" rpy="0 0 1.5708"/>
+     <geometry>
+       <mesh filename="package://smilodon_description/meshes/smilodon_collision.dae" scale="1 1 1"/>
+     </geometry>
+   </collision>
+ </link>
+   <joint name="$(arg namespace)/base_joint" type="fixed">
+    <origin xyz="0 0 0" rpy="0 0 0"/>  <!-- X-fwd, Y-lft, Z-up (ick!) -->
+    <parent link="$(arg namespace)/dummy_link"/>
+    <child link="$(arg namespace)/base_link"/>
+  </joint>
+ <gazebo>
+   <plugin name="uuv_plugin" filename="libuuv_underwater_object_ros_plugin.so">
+     <!-- Hydro parameters for the vehicle-->
+     <fluid_density>1028.0</fluid_density>
+     <flow_velocity_topic>hydrodynamics/current_velocity</flow_velocity_topic>
+     <debug>$(arg debug)</debug>
+     <link name="$(arg namespace)/base_link">
+       <neutrally_buoyant>1</neutrally_buoyant>
+       <!-- Volume, see p.31 in Berg2012 -->
+       <volume>1.8382</volume>
+       <box>
+         <width>1.5</width>
+         <length>2.6</length>
+         <height>1.6</height>
+       </box>
+       <!--
+	   Center of buoyancy according to eq. (3.1) p. 28 in Berg2012.
+	   The original values, [0.0822, -0.00773, 0.3872] however, seem to
+	   assume NWU (otherwise cob is below cog?).
+       -->
+       <center_of_buoyancy>0.0 0.0 0.3</center_of_buoyancy>
+       <hydrodynamic_model>
+         <type>fossen</type>
+         <!-- Added mass: see p.28 in Berg2012 -->
+         <added_mass>
+           779.79 -6.8773 -103.32  8.5426 -165.54 -7.8033
+           -6.8773    1222   51.29  409.44 -5.8488  62.726
+           -103.32   51.29  3659.9  6.1112 -386.42  10.774
+           8.5426  409.44  6.1112   534.9 -10.027  21.019
+           -165.54 -5.8488 -386.42 -10.027  842.69 -1.1162
+           -7.8033  62.726  10.775  21.019 -1.1162  224.32
+         </added_mass>
+         <!-- Linear damping: see p.31 in Berg2012 -->
+         <linear_damping>
+           -74.82 -69.48 -728.4 -268.8 -309.77 -105
+         </linear_damping>
+         <!-- Non-linear damping: see p.30 in Berg2012 -->
+         <quadratic_damping>
+           -748.22 -992.53 -1821.01 -672 -774.44 -523.27
+         </quadratic_damping>
+       </hydrodynamic_model>
+     </link>
+   </plugin>
+ </gazebo>
+ <gazebo>
+   <plugin name="gazebo_ros_control" filename="libgazebo_ros_control.so">
+     <robotNamespace>/$(arg namespace)</robotNamespace>
+     <robotParam>/$(arg namespace)/robot_description</robotParam>
+   </plugin>
+ </gazebo>
+ <!-- Define thrusters for propulsion -->
+ <xacro:property name="prop_mesh_file" value="file://$(find uuv_descriptions)/meshes/prop.dae"/>
+ <!-- Common values, colors, converstion, standard shapes/inertia etc.
+      Dependency for the thruster_snippets.xacro-->
+ <xacro:include filename="$(find uuv_descriptions)/urdf/common.urdf.xacro"/>
+ <!-- Various thruster models -->
+ <xacro:include filename="$(find uuv_gazebo_ros_plugins)/urdf/thruster_snippets.xacro"/>
+ <xacro:property name="prop_mesh_file" value="file://$(find uuv_descriptions)/meshes/prop.dae"/>
+ <!-- Thruster joint and link snippet
+      Wrapper for the the thruster_module_first_order_basic_fcn_macro
+      defined in uuv_gazebo_ros_plugins/urdf/thruster_snippet.
+      Uses the "thruster_cf_basic_macro"
+        1) Basic curve
+	Input: x
+	Output: thrust
+	Function: thrust = rotorConstant * x * abs(x)
+ -->
+ <xacro:macro name="thruster_macro"
+	      params="thruster_id *origin">
+   <xacro:thruster_module_first_order_basic_fcn_macro
+       namespace="$(arg namespace)"
+       thruster_id="${thruster_id}"
+       mesh_filename="${prop_mesh_file}"
+       dyn_time_constant="0.05"
+       rotor_constant="0.00031">
+     <xacro:insert_block name="origin"/>
+   </xacro:thruster_module_first_order_basic_fcn_macro>
+ </xacro:macro>
+ <!-- Port-Aft -->
+ <xacro:thruster_macro thruster_id="0">
+   <origin xyz="-3.3 0.8 -0.1" rpy="${0*d2r} ${0*d2r} ${200.0*d2r}"/>
+ </xacro:thruster_macro>
+ <!-- Stbd-Aft -->
+ <xacro:thruster_macro thruster_id="1">
+   <origin xyz="-3.3 -0.8 -0.1" rpy="${0*d2r} ${0*d2r} ${160.0*d2r}"/>
+ </xacro:thruster_macro>
+ <!-- Port-Vert -->
+ <xacro:thruster_macro thruster_id="2">
+   <origin xyz="1.8 0.8 0.4" rpy="${0*d2r} ${-110.0*d2r} ${90.0*d2r}"/>
+ </xacro:thruster_macro>
+  <!-- Stbd-Vert -->
+ <xacro:thruster_macro thruster_id="3">
+   <origin xyz="1.8 -0.8 0.4" rpy="${0*d2r} ${-110*d2r} ${-90.0*d2r}"/>
+ </xacro:thruster_macro>
+  <!-- Port-Lat -->
+ <xacro:thruster_macro thruster_id="4">
+   <origin xyz="1.8 1.3 -0.07" rpy="${0*d2r} ${0*d2r} ${90.0*d2r}"/>
+ </xacro:thruster_macro>
+   <!-- Stbd-Lat -->
+ <xacro:thruster_macro thruster_id="5">
+   <origin xyz="1.8 -1.3 -0.07" rpy="${0*d2r} ${0*d2r} ${-90.0*d2r}"/>
+ </xacro:thruster_macro>
+ <!-- Default joint state publisher -->
+ <gazebo>
+   <plugin name="uuv_joint_state_publisher" filename="libuuv_joint_state_publisher.so">
+     <robotNamespace>$(arg namespace)</robotNamespace>
+     <updateRate>50</updateRate>
+   </plugin>
+ </gazebo>
 </robot>
