Commit message: change remainder refences rov_hil to x3_sim

File: unused/urdf/macros.xacro (robot description, xacro)
@@ -253,5 +253,5 @@
 	<xacro:include filename="$(find uuv_gazebo_ros_plugins)/urdf/thruster_snippets.xacro"/>
 	<!-- thruster model -->
-	<xacro:property name="thruster_mesh_file" value="file://$(find rov_hil)/models/x3_low_poly_propeller.dae"/>
+	<xacro:property name="thruster_mesh_file" value="file://$(find x3_sim)/models/x3_low_poly_propeller.dae"/>
 	<xacro:macro name="thruster_macro" params="thruster_id *origin">
 		<xacro:thruster_module_first_order_basic_fcn_macro

File: unused/urdf/x3_v3.xacro (robot description, xacro)
@@ -2,7 +2,7 @@
 <robot name="x3_rov" xmlns:xacro="http://www.ros.org/wiki/xacro">
 	<!-- includes -->
-	<!-- <xacro:include filename="$(find rov_hil)/urdf/materials.xacro" /> -->
+	<!-- <xacro:include filename="$(find x3_sim)/urdf/materials.xacro" /> -->
 	<!-- <xacro:include filename="$(find uuv_descriptions)/urdf/common.urdf.xacro"/> -->
-	<xacro:include filename="$(find rov_hil)/urdf/macros.xacro" />
+	<xacro:include filename="$(find x3_sim)/urdf/macros.xacro" />
 	<!-- properties/variables -->
 	<xacro:arg name="debug" default="0"/>
@@ -45,5 +45,5 @@
 			<geometry>
 				<!-- <box size="${x3_length*5/8} ${x3_width * 3/5} ${x3_height}"/> -->
-				<!-- <mesh filename="package://rov_hil/models/x3_low_poly_smoothed.dae"/> -->
+				<!-- <mesh filename="package://x3_sim/models/x3_low_poly_smoothed.dae"/> -->
 				<box size="${x3_length} ${x3_width} ${x3_height}"/>
 			</geometry>

File: urdf/macros2.xacro (robot description, xacro)
@@ -246,5 +246,5 @@
 	<xacro:include filename="$(find uuv_gazebo_ros_plugins)/urdf/thruster_snippets.xacro"/>
 	<!-- Thruster model -->
-	<xacro:property name="thruster_mesh_file" value="file://$(find rov_hil)/models/x3_low_poly_propeller.dae"/>
+	<xacro:property name="thruster_mesh_file" value="file://$(find x3_sim)/models/x3_low_poly_propeller.dae"/>
 	<!-- Wrapper for thruster macro -->
 	<xacro:macro name="thruster_macro" params="thruster_id *origin">

File: urdf/x3_components.xacro (robot description, xacro)
@@ -2,5 +2,5 @@
 <robot name="x3_components" xmlns:xacro="http://www.ros.org/wiki/xacro">
 	<!-- includes -->
-	<xacro:include filename="$(find rov_hil)/urdf/helpers.xacro" />
+	<xacro:include filename="$(find x3_sim)/urdf/helpers.xacro" />
 	<!-- properties/variables -->
 	<xacro:arg name="debug" default="0"/>
@@ -54,5 +54,5 @@
 	<xacro:include filename="$(find uuv_gazebo_ros_plugins)/urdf/thruster_snippets.xacro"/>
 	<!-- Thruster model -->
-	<xacro:property name="thruster_mesh_file" value="file://$(find rov_hil)/models/x3_low_poly_propeller.dae"/>
+	<xacro:property name="thruster_mesh_file" value="file://$(find x3_sim)/models/x3_low_poly_propeller.dae"/>
 	<!-- Wrapper for thruster macro -->
 	<xacro:macro name="thruster_macro" params="thruster_id *origin">

File: urdf/x3_sensors.xacro (robot description, xacro)
@@ -2,5 +2,5 @@
 <robot name="x3_sensors" xmlns:xacro="http://www.ros.org/wiki/xacro">
 	<!-- includes -->
-	<xacro:include filename="$(find rov_hil)/urdf/helpers.xacro" />
+	<xacro:include filename="$(find x3_sim)/urdf/helpers.xacro" />
 	<!-- properties/variables -->
 	<xacro:arg name="debug" default="0"/>

File: urdf/x3_v2.xacro (robot description, xacro)
@@ -2,6 +2,6 @@
 <robot name="x3_rov" xmlns:xacro="http://www.ros.org/wiki/xacro">
 	<!-- includes -->
-	<!-- <xacro:include filename="$(find rov_hil)/urdf/materials.xacro" /> -->
-	<xacro:include filename="$(find rov_hil)/urdf/macros2.xacro" />
+	<!-- <xacro:include filename="$(find x3_sim)/urdf/materials.xacro" /> -->
+	<xacro:include filename="$(find x3_sim)/urdf/macros2.xacro" />
 	<!-- properties/variables -->
 	<xacro:arg name="debug" default="0"/>
@@ -43,5 +43,5 @@
 			<geometry>
 				<!-- <box size="${x3_length*5/8} ${x3_width * 3/5} ${x3_height}"/> -->
-				<mesh filename="package://rov_hil/models/x3_low_poly_smoothed.dae"/>
+				<mesh filename="package://x3_sim/models/x3_low_poly_smoothed.dae"/>
 			</geometry>
 			<material name="grey"/>

File: urdf/x3_v3.xacro (robot description, xacro)
@@ -2,8 +2,8 @@
 <robot name="x3_rov" xmlns:xacro="http://www.ros.org/wiki/xacro">
 	<!-- includes -->
-	<!-- <xacro:include filename="$(find rov_hil)/urdf/materials.xacro" /> -->
-	<xacro:include filename="$(find rov_hil)/urdf/helpers.xacro" />
-	<xacro:include filename="$(find rov_hil)/urdf/x3_components.xacro" />
-	<xacro:include filename="$(find rov_hil)/urdf/x3_sensors.xacro" />
+	<!-- <xacro:include filename="$(find x3_sim)/urdf/materials.xacro" /> -->
+	<xacro:include filename="$(find x3_sim)/urdf/helpers.xacro" />
+	<xacro:include filename="$(find x3_sim)/urdf/x3_components.xacro" />
+	<xacro:include filename="$(find x3_sim)/urdf/x3_sensors.xacro" />
 	<!-- properties/variables -->
 	<xacro:arg name="debug" default="0"/>
@@ -49,5 +49,5 @@
 			<geometry>
 				<!-- <box size="${x3_length*5/8} ${x3_width * 3/5} ${x3_height}"/> -->
-				<mesh filename="package://rov_hil/models/x3_low_poly_smoothed.dae"/>
+				<mesh filename="package://x3_sim/models/x3_low_poly_smoothed.dae"/>
 			</geometry>
 			<material name="grey"/>
